Commit message: working sim with arm and gripper control and movement api

File: urdf/ur12e_with_gripper.urdf (robot description, URDF)
Before this commit: robot ur12e_with_gripper, 24 links, 23 joints
Links:
- removed link left_inner_finger
- removed link left_inner_finger_pad
- removed link left_inner_knuckle
- removed link left_outer_finger
- removed link left_outer_knuckle
- removed link right_inner_finger
- removed link right_inner_finger_pad
- removed link right_inner_knuckle
- removed link right_outer_finger
- removed link right_outer_knuckle
- removed link robotiq_arg2f_base_link
- added link robotiq_85_base_link, mass 6.6320197e-01; collision mesh filename=file:///opt/ros/kilted/share/robotiq_description/meshes/col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; visual mesh filename=file:///opt/ros/kilted/share/robotiq_description/meshes/vis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
- added link robotiq_85_left_finger_link, mass 4.260376752e-02; collision mesh filename=file:///opt/ros/kilted/share/robotiq_description/meshes/col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; visual mesh filename=file:///opt/ros/kilted/share/robotiq_description/meshes/vis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
- added link robotiq_85_left_finger_tip_link, mass 4.268588744e-02; collision mesh filename=file:///opt/ros/kilted/share/robotiq_description/meshes/col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; visual mesh filename=file:///opt/ros/kilted/share/robotiq_description/meshes/vis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
- added link robotiq_85_left_inner_knuckle_link, mass 2.969376448e-02; collision mesh filename=file:///opt/ros/kilted/share/robotiq_description/meshes/col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; visual mesh filename=file:///opt/ros/kilted/share/robotiq_description/meshes/vis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
- added link robotiq_85_left_knuckle_link, mass 1.384773208e-02; collision mesh filename=file:///opt/ros/kilted/share/robotiq_description/meshes/col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; visual mesh filename=file:///opt/ros/kilted/share/robotiq_description/meshes/vis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
- added link robotiq_85_right_finger_link, mass 4.260376752000000e-02; collision mesh filename=file:///opt/ros/kilted/share/robotiq_description/meshes/col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; visual mesh filename=file:///opt/ros/kilted/share/robotiq_description/meshes/vis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
- added link robotiq_85_right_finger_tip_link, mass 4.268588744e-02; collision mesh filename=file:///opt/ros/kilted/share/robotiq_description/meshes/col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; visual mesh filename=file:///opt/ros/kilted/share/robotiq_description/meshes/vis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
- added link robotiq_85_right_inner_knuckle_link, mass 2.969376448e-02; collision mesh filename=file:///opt/ros/kilted/share/robotiq_description/meshes/col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; visual mesh filename=file:///opt/ros/kilted/share/robotiq_description/meshes/vis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
- added link robotiq_85_right_knuckle_link, mass 1.384773208e-02; collision mesh filename=file:///opt/ros/kilted/share/robotiq_description/meshes/col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; visual mesh filename=file:///opt/ros/kilted/share/robotiq_description/meshes/vis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
Joints:
- removed joint finger_joint
- removed joint left_inner_finger_joint
- removed joint left_inner_finger_pad_joint
- removed joint left_inner_knuckle_joint
- removed joint left_outer_finger_joint
- removed joint right_inner_finger_joint
- removed joint right_inner_finger_pad_joint
- removed joint right_inner_knuckle_joint
- removed joint right_outer_finger_joint
- removed joint right_outer_knuckle_joint
- removed joint robotiq_2f_gripper_fix
- added joint robotiq_85_base_joint: type fixed, parent tool0, child robotiq_85_base_link, origin xyz=0 0 0 rpy=0 0 0
- added joint robotiq_85_left_finger_joint: type fixed, parent robotiq_85_left_knuckle_link, child robotiq_85_left_finger_link, origin xyz=0.03152616 0.0 -0.00376347 rpy=0 0 0
- added joint robotiq_85_left_finger_tip_joint: type continuous, parent robotiq_85_left_finger_link, child robotiq_85_left_finger_tip_link, origin xyz=0.00563134 0.0 0.04718515 rpy=0 0 0, axis 0 -1 0, mimic joint=robotiq_85_left_knuckle_joint multiplier=-1
- added joint robotiq_85_left_inner_knuckle_joint: type continuous, parent robotiq_85_base_link, child robotiq_85_left_inner_knuckle_link, origin xyz=0.0127 0.0 0.06142 rpy=0 0 0, axis 0 -1 0, mimic joint=robotiq_85_left_knuckle_joint
- added joint robotiq_85_left_knuckle_joint: type revolute, parent robotiq_85_base_link, child robotiq_85_left_knuckle_link, origin xyz=0.03060114 0.0 0.05490452 rpy=0 0 0, axis 0 -1 0, limit lower=0.0 upper=0.8 effort=50 velocity=0.5
- added joint robotiq_85_right_finger_joint: type fixed, parent robotiq_85_right_knuckle_link, child robotiq_85_right_finger_link, origin xyz=-0.03152616 0.0 -0.00376347 rpy=0 0 0
- added joint robotiq_85_right_finger_tip_joint: type continuous, parent robotiq_85_right_finger_link, child robotiq_85_right_finger_tip_link, origin xyz=-0.00563134 0.0 0.04718515 rpy=0 0 0, axis 0 -1 0, mimic joint=robotiq_85_left_knuckle_joint
- added joint robotiq_85_right_inner_knuckle_joint: type continuous, parent robotiq_85_base_link, child robotiq_85_right_inner_knuckle_link, origin xyz=-0.0127 0.0 0.06142 rpy=0 0 0, axis 0 -1 0, mimic joint=robotiq_85_left_knuckle_joint multiplier=-1
- added joint robotiq_85_right_knuckle_joint: type revolute, parent robotiq_85_base_link, child robotiq_85_right_knuckle_link, origin xyz=-0.03060114 0.0 0.05490452 rpy=0 0 0, axis 0 -1 0, limit lower=-0.8 upper=0.0 effort=50 velocity=0.5, mimic joint=robotiq_85_left_knuckle_joint multiplier=-1
